File: phantom_3_pro_gimbal_top_board/phantom_3_pro_gimbal_top_board.sch (KiCad schematic (older format))
At the start: 79 parts

Commit message: Gimbal Top: Better symbols, dc-dc circuits
Symbols were updated so that pins match to footpints.
More footprints added.
Switching regulator circuits were drawn based on application examples.
Parts:
- removed TP? (x2): 3.3VD, symbol TEST
- removed TP?: VDDA, symbol TEST
- removed TP?: VDD, symbol TEST
- removed TP?: A9S_3.3VD, symbol TEST
- removed TP?: ﻿3V3VD, symbol TEST
- removed TP?: 1.8VD, symbol TEST
- removed TP?: 1V2, symbol TEST
- removed TP?: 12V, symbol TEST
- removed TP?: +5V, symbol TEST
- removed TP?: VCC3V3, symbol TEST
- removed TP?: VCC1V8, symbol TEST
- removed TP?: 1.25DDR2, symbol TEST
- removed TP?: BT01, symbol TEST
- removed TP?: MB, symbol TEST
- removed TP? (x7): GND, symbol TEST
- removed TP?: MA, symbol TEST
- removed TP?: BT00, symbol TEST
- removed TP?: H2, symbol TEST
- removed TP?: MC, symbol TEST
- removed TP?: TDO, symbol TEST
- removed TP?: H1, symbol TEST
- removed TP?: B_S, symbol TEST
- removed TP?: U3_CX, symbol TEST
- removed TP?: H3, symbol TEST
- removed TP?: MCLR_N, symbol TEST
- removed TP?: 365, symbol TEST
- removed TP?: TMS, symbol TEST
- removed TP?: U3_RX, symbol TEST
- removed TP?: U1RT, symbol TEST
- removed TP?: BOOT0, symbol TEST
- removed TP?: TDI, symbol TEST
- removed TP?: U1TT, symbol TEST
- removed TP?: OUT6, symbol TEST
- removed TP?: CLK, symbol TEST
- removed TP?: DM-, symbol TEST
- removed TP?: MOSI, symbol TEST
- removed TP?: PGED, symbol TEST
- removed TP?: OUT8, symbol TEST
- removed TP?: 368_U0_RXP, symbol TEST
- removed TP?: DP+, symbol TEST
- removed TP?: URAT2_TX, symbol TEST
- removed TP?: SWDIO, symbol TEST
- removed TP?: CS_DSP, symbol TEST
- removed TP?: PGEC, symbol TEST
- removed TP?: U1_T1, symbol TEST
- removed TP?: CANH, symbol TEST
- removed TP?: U0_R, symbol TEST
- removed TP?: RST, symbol TEST
- removed TP?: CANL, symbol TEST
- removed TP?: URAT2_RX, symbol TEST
- removed TP?: 368_U0_TXP, symbol TEST
- removed TP?: SCL_DSP, symbol TEST
- removed TP?: U0_T, symbol TEST
- removed TP?: SWCLK, symbol TEST
- removed TP?: RSTEX, symbol TEST
- removed TP?: GIMBAL, symbol TEST
- removed TP?: U1_R1, symbol TEST
- removed U?: TMS320DM365_ZCE_338_A, symbol TMS320DM365_ZCE_338_A-RESCUE-phantom_3_pro_gimbal_top_board
- removed U?: TMS320DM365_ZCE_338_B, symbol TMS320DM365_ZCE_338_B-RESCUE-phantom_3_pro_gimbal_top_board
- removed U?: TMS320DM365_ZCE_338_C, symbol TMS320DM365_ZCE_338_C-RESCUE-phantom_3_pro_gimbal_top_board
- removed U?: TMS320DM365_ZCE_338_D, symbol TMS320DM365_ZCE_338_D-RESCUE-phantom_3_pro_gimbal_top_board
- removed U?: TLV62130, symbol TLV62130
- added C1, C10, C12, C17, C19, C24, C25, C27, C29, C5: 10uF?, symbol C_Small
- added C11, C13, C18, C20: xuF?, symbol C_Small
- added C14, C21: 470nF?, symbol C_Small
- added C15, C16, C22, C32, C33, C34, C9: 1uF?, symbol C_Small
- added C2, C26, C28, C6: 100nF?, symbol C_Small
- added C23: 22pF?, symbol C_Small
- added C3, C7: 3.3nF?, symbol C_Small
- added C30, C31: 2.2uF?, symbol C_Small
- added C4, C8: 22uF?, symbol C_Small
- added D1, D2, D3: MBR0540, symbol D_Small_ALT
- added L1, L2, L3, L4, L5: 2.2uH, Inductors_SMD:L_Vishay_IHLP-1212, symbol L_Small
- added R1, R4, R7: 100kΩ?, symbol R_Small
- added R10, R11, R12, R13, R14, R15, R2, R3, R5, R6, R8, R9: xΩ?, symbol R_Small
- added R16, R17: 475kΩ?, symbol R_Small
- added R18: 976kΩ?, symbol R_Small
- added R19, R20, R22: 47kΩ?, symbol R_Small
- added R21: 232kΩ?, symbol R_Small
- added R23: 22Ω?, symbol R_Small
- added R24, R25: 5.1kΩ?, symbol R_Small
- added R26: 470Ω?, symbol R_Small
- added R27: 1.1kΩ?, symbol R_Small
- added TP1: CS_DSP, symbol TEST
- added TP10: TDI, symbol TEST
- added TP11: PGED, symbol TEST
- added TP12: PGEC, symbol TEST
- added TP13: SWCLK, symbol TEST
- added TP14: TDO, symbol TEST
- added TP15: MCLR_N, symbol TEST
- added TP16: BOOT0, symbol TEST
- added TP17: MOSI, symbol TEST
- added TP18: SWDIO, symbol TEST
- added TP19: RST, symbol TEST
- added TP2: SCL_DSP, symbol TEST
- added TP20: RSTEX, symbol TEST
- added TP21: BT01, symbol TEST
- added TP22: BT00, symbol TEST
- added TP23: MC, symbol TEST
- added TP24: B_S, symbol TEST
- added TP25: 365, symbol TEST
- added TP26: OUT6, symbol TEST
- added TP27: OUT8, symbol TEST
- added TP28: GIMBAL, symbol TEST
- added TP29: CLK, symbol TEST
- added TP3: U0_R, symbol TEST
- added TP30: U1_T1, symbol TEST
- added TP31: U1_R1, symbol TEST
- added TP32: 12V, symbol TEST
- added TP33: +5V, symbol TEST
- added TP34: CANH, symbol TEST
- added TP35: CANL, symbol TEST
- added TP36, TP39: 3.3VD, symbol TEST
- added TP37: A9S_3.3VD, symbol TEST
- added TP38: ﻿3V3VD, symbol TEST
- added TP4: U0_T, symbol TEST
- added TP40: VCC3V3, symbol TEST
- added TP41: 1.8VD, symbol TEST
- added TP42: VCC1V8, symbol TEST
- added TP43: MB, symbol TEST
- added TP44: MA, symbol TEST
- added TP45: H2, symbol TEST
- added TP46: H1, symbol TEST
- added TP47: H3, symbol TEST
- added TP48: U1RT, symbol TEST
- added TP49: U1TT, symbol TEST
- added TP5: U3_CX, symbol TEST
- added TP50: URAT2_TX, symbol TEST
- added TP51: URAT2_RX, symbol TEST
- added TP52: VDDA, symbol TEST
- added TP53: VDD, symbol TEST
- added TP54: 1V2, symbol TEST
- added TP55: 1.25DDR2, symbol TEST
- added TP56, TP57, TP58, TP59, TP60, TP61, TP62: GND, symbol TEST
- added TP6: U3_RX, symbol TEST
- added TP63: 368_U0_RXP, symbol TEST
- added TP64: 368_U0_TXP, symbol TEST
- added TP7: DM-, symbol TEST
- added TP8: DP+, symbol TEST
- added TP9: TMS, symbol TEST
- added U1: TMS320DM365_ZCE_338, Housings_BGA-v2:PBGA-N338_19x19_13x13mm_Pitch0.65mm, symbol TMS320DM365_ZCE_338
- added U7: SN74AVC8T245RHL, symbol SN74AVC8T245RHL
- added U9: TLV62130, Housings_DFN_QFN:QFN-16-1EP_3x3mm_Pitch0.5mm_ThermalVias, symbol TLV62130
- U10: renamed from U?; footprint (none) -> Housings_DFN_QFN:QFN-24-1EP_4x4mm_Pitch0.5mm
- U11: renamed from U?; footprint (none) -> Housings_DFN_QFN-v2:QFN-20_3x3mm_Pitch0.4mm_NoMask
- U5: renamed from U?; footprint TW-BGA-84 -> Housings_BGA-v2:BGA-84_2x3x15_8.0x12.5mm_Pitch0.8mm
- U6: renamed from U?; footprint (none) -> Housings_DFN_QFN:QFN-16-1EP_3x3mm_Pitch0.5mm_ThermalVias
- U8: renamed from U?; footprint FBGA-168 -> Housings_BGA-v2:UFBGA-168_12x12mm_Pitch0.5mm
- gave numbers to parts that had none: 5
Connections:
- net labels added: EN_1.2, EN_1.8, EN_3.3, GND, SYS_EN, VIN, VOUT_1.2, VOUT_1.8, VOUT_3.3, nManRst
- wire segments 0 -> 177
Other:
- moved on the sheet: TP10, U10, U11, U5, U6
