File: phantom_3_pro_gimbal_top_board/phantom_3_pro_gimbal_top_board.sch (KiCad schematic (older format))
At the start: 146 parts, among them J1 CONN_OFDM, J2 CONN_ARMS2, J3 CONN_ARMS1, J4 CONN_CENTER, U1 TMS320DM365_ZCE_338, U10 LM26480-Q1_WQFN_24, U11 TPS650061_RUK_20, U5 IS43DR16640B, U6 TLV62130, U7 SN74AVC8T245RHL, U8 EDB8132B3PB_DDR2_RAM, U9 TLV62130, Y1 Crystal_GND23_Small

Commit message: Gimbal Top: Measured and filled part of DC-DC conv
Checked part of voltage regulator circuits with multimeter.
Associated a few footprints with schematic, updated values.
Parts:
- added C35, C36: 22uF?, Capacitors_SMD:C_1206, symbol C_Small
- added C37, C38: 2.2uF?, Capacitors_SMD:C_0603, symbol C_Small
- added C39, C40, C42: 100nF?, Capacitors_SMD:C_0603, symbol C_Small
- added C41, C43: 10nF?, Capacitors_SMD:C_0603, symbol C_Small
- added C44: 100pF?, Capacitors_SMD:C_0402, symbol C_Small
- added TP65: GND, Measurement_Points:Measurement_Point_Round-SMD-Pad_Small, symbol TEST
- C1: footprint (none) -> Capacitors_SMD:C_0805
- C2, C34: footprint (none) -> Capacitors_SMD:C_0402
- C23: value 22pF? -> 22pF; footprint (none) -> Capacitors_SMD:C_0402
- C27, C29: value 10uF? -> 10nF?; footprint (none) -> Capacitors_SMD:C_0402
- C30: footprint (none) -> Capacitors_SMD:C_0603
- C4, C8: value 22uF? -> 2.2uF?; footprint (none) -> Capacitors_SMD:C_1206
- L5: footprint Inductors_SMD:L_Vishay_IHLP-1212 -> Inductors_SMD:L_Neosid_SMS-ME3010
- R16, R17: value 475kΩ? -> 220kΩ; footprint (none) -> Resistors_SMD:R_0402
- R18: value 976kΩ? -> 1kΩ; footprint (none) -> Resistors_SMD:R_0402
- R20: value 47kΩ? -> 50kΩ; footprint (none) -> Resistors_SMD:R_0402
- R27: value 1.1kΩ? -> 2kΩ; footprint (none) -> Resistors_SMD:R_0402
- R5, R6: value xΩ? -> 2.8kΩ; footprint (none) -> Resistors_SMD:R_0402
- TP1, TP10, TP11, TP12, TP13, TP14, TP15, TP16, TP17, TP18, TP19, TP2, TP20, TP21, TP22, TP23, TP24, TP25, TP26, TP27, TP28, TP29, TP3, TP30, TP31, TP32, TP33, TP34, TP35, TP36, TP37, TP38, TP39, TP4, TP40, TP41, TP42, TP43, TP44, TP45, TP46, TP47, TP48, TP49, TP5, TP50, TP51, TP52, TP53, TP54, TP55, TP56, TP57, TP58, TP59, TP6, TP60, TP61, TP62, TP63, TP64, TP7, TP8, TP9: footprint (none) -> Measurement_Points:Measurement_Point_Round-SMD-Pad_Small
- U11: value TPS650061_RUK_20 -> TPS650061
Connections:
- net labels added: +5V, 12V, VCC1V2, VCC1V8, VCC3V3, VDD1V6
- net labels removed: VIN, VOUT_1.2, VOUT_1.8, VOUT_3.3
- wire segments 177 -> 277
Other:
- moved on the sheet: C1, C27, C29, C4, C8, R19

Commit message: Gimbal Top: Added more symbols and footprints.
Parts:
- added J5: USB_OTG, Connectors:USB_Micro-B, symbol USB_OTG
- added J6: CONN_01X02, symbol CONN_01X02
- added J7: CONN_MOTOR, Connectors_FFC:Flat_Foam_Conn-ZIF-14S-0.5H_14x0.50mm_Angled, symbol CONN_01X14
- added J8: Micro_SD_Card, Connectors:microSD_Card_Receptacle_Wuerth_693072010801, symbol Micro_SD_Card
- added Q1: PMBT3904, TO_SOT_Packages_SMD:SOT-23, symbol Q_NPN_BEC
- added U12: MLX90316, Housings_SOIC:SOIC-8-1EP_3.9x4.9mm_Pitch1.27mm, symbol MLX90316
- added U13: NCP585, TO_SOT_Packages_SMD-v2:SOT-25, symbol NCP585
- added U14, U15: TS3USB221A-Q1, texas-var-geda:RSE10, symbol TS3USB221A-Q1
- added U16: dsPIC33EP128MC504, Housings_LGA-v2:VTLA-44_LGA-44_6x6mm_Pitch0.5mm, symbol dsPIC33EPxxxMC50x
- added U2: STM32F407IGH6, Housings_BGA-v2:UFBGA176p25-10x10mm_pitch0.65mm, symbol STM32F4XXH1
- added U3: MT29F1G08, Housings_BGA-v2:VFBGA-63_11x9_9.0x7.4mm_Pitch0.8mm, symbol MT29F1G08
- added U4: MT29F2G08, Housings_BGA-v2:VFBGA-63_11x9_9.0x7.4mm_Pitch0.8mm, symbol MT29F2G08
- J1: value CONN_OFDM -> CONN_CENTER; footprint (none) -> Connectors_Hirose:Hirose_DF13C-08P-1.25V_08x1.25mm_Straight
- J2, J3: footprint (none) -> Connectors_FFC:Flat_Foam_Conn-ZIF-35D-0.6H_35x0.60mm_Angled
- J4: value CONN_CENTER -> CONN_OFDM; footprint (none) -> Connectors_Hirose:Hirose_DF13C-06P-1.25V_06x1.25mm_Straight
- R5, R6: value 2.8kΩ -> 2.8kΩ?
- TP38: value ﻿3V3VD -> 3V3VD
- U1: value TMS320DM365_ZCE_338 -> TMS320DM365ZCE
- U10: value LM26480-Q1_WQFN_24 -> LM26480
- U7: footprint (none) -> Housings_DFN_QFN-v2:RHL0024_PVQFN-n24p4_4.3x6.3mm_Pitch0.5mm
- U8: value EDB8132B3PB_DDR2_RAM -> EDB8132B3PB
Connections:
- net labels added: VDD1V1, VDDA1V1
- net labels removed: VDD1V6
- wire segments 277 -> 216
Other:
- moved on the sheet: C35, C36, J1, J2, J3, J4, Y1

Commit message: Gimbal Top: Drawn USB circuits, and USB mux'es.
USB multiplexers are used for both USB outputs, though
connected in very different ways.
Parts:
- added R28, R30: ∞Ω, symbol R_Small
- added R29, R31, R32, R33: 0Ω, Resistors_SMD:R_0402, symbol R_Small
- added R34: ∞Ω, Resistors_SMD:R_0402, symbol R_Small
- added R35, R36: 4.7kΩ, Resistors_SMD:R_0402, symbol R_Small
- added R37: 800kΩ, symbol R_Small
- added R38: 0.3Ω, symbol R_Small
- added U17: MAX3051EKA_to_verify, symbol PCA82C251
- renumbered U15 to U14, U14 to U15
Connections:
- net labels added: 3.3VD, CANH, CANL
- wire segments 216 -> 248
Other:
- note added: "to\nAmbarella"
- note added: "to\nDaVinci"
- moved on the sheet: J4, J5, Q1, U14, U15

Commit message: Gimbal/ESC Center: Minor updates.
Connections:
- wire segments 248 -> 249
Other:
- note added: "unknown logic sets "S"\nto high and enables USB\nafter initial boot"
Changed lines of the file:
@@
 $EndComp
 Wire Wire Line
-	19450 3650 19600 3650
+	19450 3650 19800 3650
 Wire Wire Line
 	19600 3650 19600 4000
@@
 Text Label 15550 4400 0    60   ~ 0
 CANL
+Wire Wire Line
+	19800 3650 19800 3250
+Connection ~ 19600 3650
+Text Notes 19400 3300 0    60   ~ 0
+unknown logic sets "S"\nto high and enables USB\nafter initial boot
 $EndSCHEMATC

Commit message: All: Preparing for KiCad version change.
Parts:
- J1: symbol CONN_01X08 -> Connector_Generic:Conn_01x08
- J2, J3: symbol CONN_01X35 -> Connector_Generic:Conn_01x35
- J4: symbol CONN_01X06 -> Connector_Generic:Conn_01x06
- J6: symbol CONN_01X02 -> Connector_Generic:Conn_01x02
- J7: symbol CONN_01X14 -> Connector_Generic:Conn_01x14
- TP1, TP10, TP11, TP12, TP13, TP14, TP15, TP16, TP17, TP18, TP19, TP2, TP20, TP21, TP22, TP23, TP24, TP25, TP26, TP27, TP28, TP29, TP3, TP30, TP31, TP32, TP33, TP34, TP35, TP36, TP37, TP38, TP39, TP4, TP40, TP41, TP42, TP43, TP44, TP45, TP46, TP47, TP48, TP49, TP5, TP50, TP51, TP52, TP53, TP54, TP55, TP56, TP57, TP58, TP59, TP6, TP60, TP61, TP62, TP63, TP64, TP65, TP7, TP8, TP9: symbol TEST -> Connector:TestPoint

Commit message: Overview: Upgraded to KiCAD 5.0.1.
Parts:
- removed J5: USB_OTG, Connectors:USB_Micro-B, symbol USB_OTG
- removed J8: Micro_SD_Card, Connectors:microSD_Card_Receptacle_Wuerth_693072010801, symbol Micro_SD_Card
- added J5: USB_OTG, Connectors:USB_Micro-B, symbol Connector:USB_OTG
- added J8: Micro_SD_Card, symbol Connector:Micro_SD_Card
- C1, C10, C11, C12, C13, C14, C15, C16, C17, C18, C19, C2, C20, C21, C22, C23, C24, C25, C26, C27, C28, C29, C3, C30, C31, C32, C33, C34, C35, C36, C37, C38, C39, C4, C40, C41, C42, C43, C44, C5, C6, C7, C8, C9: symbol C_Small -> Device:C_Small
- D1, D2, D3: symbol D_Small_ALT -> Device:D_Small_ALT
- L1, L2, L3, L4, L5: symbol L_Small -> Device:L_Small
- Q1: symbol Q_NPN_BEC -> Device:Q_NPN_BEC
- R1, R10, R11, R12, R13, R14, R15, R16, R17, R18, R19, R2, R20, R21, R22, R23, R24, R25, R26, R27, R28, R29, R3, R30, R31, R32, R33, R34, R35, R36, R37, R38, R4, R5, R6, R7, R8, R9: symbol R_Small -> Device:R_Small
- U1: symbol TMS320DM365_ZCE_338 -> texas-uc:TMS320DM365_ZCE_338
- U10: symbol LM26480-Q1_WQFN_24 -> regul-v2:LM26480-Q1_WQFN_24
- U11: symbol TPS650061_RUK_20 -> regul-v2:TPS650061_RUK_20
- U12: symbol MLX90316 -> sensors-v2:MLX90316
- U13: symbol NCP585 -> regul-v2:NCP585
- U14, U15: symbol TS3USB221A-Q1 -> texas-mux:TS3USB221A-Q1
- U16: symbol dsPIC33EPxxxMC50x -> microchip-dsp:dsPIC33EPxxxMC50x
- U17: symbol PCA82C251 -> phantom_3_pro_gimbal_top_board-rescue:PCA82C251
- U2: symbol STM32F4XXH1 -> texas-uc:STM32F4XXH1
- U3: symbol MT29F1G08 -> memory-flash:MT29F1G08
- U4: symbol MT29F2G08 -> memory-flash:MT29F2G08
- U5: symbol IS43DR16640B -> memory-ram:IS43DR16640B
- U6, U9: symbol TLV62130 -> regul-v2:TLV62130
- U7: symbol SN74AVC8T245RHL -> texas-trx:SN74AVC8T245RHL
- U8: symbol EDB8132B3PB_DDR2_RAM -> memory-ram:EDB8132B3PB_DDR2_RAM
- Y1: symbol Crystal_GND23_Small -> Device:Crystal_GND23_Small
Connections:
- wire segments 249 -> 326
Other:
- moved on the sheet: J1, J4, J7

Commit message: All: Finished updating to KiCad 5.0.1.
Parts:
- U17: symbol phantom_3_pro_gimbal_top_board-rescue:PCA82C251 -> Interface_CAN_LIN:PCA82C251
Changed lines of the file:
@@
 	20250 3900 19850 3900
 $Comp
-L phantom_3_pro_gimbal_top_board-rescue:PCA82C251 U17
+L Interface_CAN_LIN:PCA82C251 U17
 U 1 1 5A280A05
 P 15100 4400
