File: phantom_3_pro_esc_center_board/phantom_3_pro_esc_center_board.sch (KiCad schematic (older format))
At the start: 138 parts, among them J1 CONN_BAT, J10 M1_BK, J11 M1_RD, J12 M1_YW, J13 M2_YW, J14 M2_RD, J15 M2_BK, J16 M3_BK, J17 M3_RD, J18 M3_YW, J19 M4_YW, J2 CONN_GPS, J20 M4_RD, J21 M4_BK, J22 CONN_BAT_PWR, J23 M1_R, J24 M1_G, J25 M2_R, J26 M2_G, J27 M1_VCC, J28 M2_VCC, J29 M3_R, J3 CONN_GIMBAL, J30 M3_G, J31 M4_R, J32 M4_G, J33 M3_VCC, J34 M4_VCC, J4 CONN_CMPAS, J5 CONN_OFDM, J6 CONN_USB, J7 CONN_API, J8 CONN_MC_FRONT, J9 CONN_MC_BACK, Q25 Q_NMOS_DGS, Q26 Q_NMOS_DGS, U1 TPS54531, U2 TPS54531, U3 LM25116

Commit message: Gimbal/ESC Center: Minor updates.
Parts:
- TP62: value OFDM TX6 -> VPS TX6
- TP65: value OFDM RX6 -> VPS RX6
Changed lines of the file:
@@
 P 4450 3150
 F 0 "TP65" H 4450 3450 50  0001 C BNN
-F 1 "OFDM RX6" H 4450 3400 50  0000 C CNN
+F 1 "VPS RX6" H 4450 3400 50  0000 C CNN
 F 2 "" H 4450 3150 50  0001 C CNN
 F 3 "" H 4450 3150 50  0001 C CNN
@@
 P 4250 2950
 F 0 "TP62" H 4250 3250 50  0001 C BNN
-F 1 "OFDM TX6" H 4250 3200 50  0000 C CNN
+F 1 "VPS TX6" H 4250 3200 50  0000 C CNN
 F 2 "" H 4250 2950 50  0001 C CNN
 F 3 "" H 4250 2950 50  0001 C CNN

Commit message: All: Preparing for KiCad version change.
Parts:
- J1, J22: symbol CONN_01X02 -> Connector_Generic:Conn_01x02
- J10, J11, J12, J13, J14, J15, J16, J17, J18, J19, J20, J21, J23, J24, J25, J26, J27, J28, J29, J30, J31, J32, J33, J34: symbol TEST_1P -> Connector:TestPoint
- J2, J4: symbol CONN_01X05 -> Connector_Generic:Conn_01x05
- J3: symbol CONN_01X08 -> Connector_Generic:Conn_01x08
- J5: symbol CONN_01X10 -> Connector_Generic:Conn_01x10
- J6, J7: symbol CONN_01X03 -> Connector_Generic:Conn_01x03
- J8: symbol CONN_01X20 -> Connector_Generic:Conn_01x20
- J9: symbol CONN_01X21 -> Connector_Generic:Conn_01x21
- TP53, TP54, TP55, TP56, TP57, TP58, TP59, TP60, TP61, TP62, TP63, TP64, TP65, TP66, TP67, TP68, TP69, TP70, TP71: symbol TEST -> Connector:TestPoint
Changed lines of the file:
@@
 $EndSheet
 $Comp
-L CONN_01X20 J8
+L Connector_Generic:Conn_01x20 J8
 U 1 1 58FEFB33
 P 2700 1900
@@
 $EndComp
 $Comp
-L CONN_01X21 J9
+L Connector_Generic:Conn_01x21 J9
 U 1 1 58FEFD57
 P 2650 2700
@@
 $EndComp
 $Comp
-L CONN_01X03 J6
+L Connector_Generic:Conn_01x03 J6
 U 1 1 58FF0F6F
 P 2400 650
@@
 $EndComp
 $Comp
-L CONN_01X10 J5
+L Connector_Generic:Conn_01x10 J5
 U 1 1 58FF110D
 P 4900 2700
@@
 $EndComp
 $Comp
-L CONN_01X02 J1
+L Connector_Generic:Conn_01x02 J1
 U 1 1 58FF3502
 P 750 850
@@
 $EndComp
 $Comp
-L CONN_01X05 J2
+L Connector_Generic:Conn_01x05 J2
 U 1 1 58FF381B
 P 1000 3150
@@
 $EndComp
 $Comp
-L CONN_01X05 J4
+L Connector_Generic:Conn_01x05 J4
 U 1 1 58FF3CA6
 P 4900 1800
@@
 $EndComp
 $Comp
-L CONN_01X08 J3
+L Connector_Generic:Conn_01x08 J3
 U 1 1 58FF3FD7
 P 3300 650
@@
 $EndComp
 $Comp
-L CONN_01X03 J7
+L Connector_Generic:Conn_01x03 J7
 U 1 1 58FF4522
 P 4900 1150
@@
 $EndComp
 $Comp
-L TEST_1P J12
+L Connector:TestPoint J12
 U 1 1 58FFAD12
 P 6750 900
@@
 $EndComp
 $Comp
-L TEST_1P J11
+L Connector:TestPoint J11
 U 1 1 58FFB359
 P 6750 800
@@
 $EndComp
 $Comp
-L TEST_1P J10
+L Connector:TestPoint J10
 U 1 1 58FFB444
 P 6750 700
@@
 $EndComp
 $Comp
-L TEST_1P J19
+L Connector:TestPoint J19
 U 1 1 58FFDAEE
 P 6750 2500
@@
 $EndComp
 $Comp
-L TEST_1P J20
+L Connector:TestPoint J20
 U 1 1 58FFDAF4
 P 6750 2600
@@
 $EndComp
 $Comp
-L TEST_1P J21
+L Connector:TestPoint J21
 U 1 1 58FFDAFA
 P 6750 2700
@@
 $EndComp
 $Comp
-L TEST_1P J13
+L Connector:TestPoint J13
 U 1 1 58FFDD88
 P 6750 1300
@@
 $EndComp
 $Comp
-L TEST_1P J14
+L Connector:TestPoint J14
 U 1 1 58FFDD8E
 P 6750 1400
@@
 $EndComp
 $Comp
-L TEST_1P J15
+L Connector:TestPoint J15
 U 1 1 58FFDD94
 P 6750 1500
@@
 $EndComp
 $Comp
-L TEST_1P J18
+L Connector:TestPoint J18
 U 1 1 58FFE004
 P 6750 2100
@@
 $EndComp
 $Comp
-L TEST_1P J17
+L Connector:TestPoint J17
 U 1 1 58FFE00A
 P 6750 2000
@@
 $EndComp
 $Comp
-L TEST_1P J16
+L Connector:TestPoint J16
 U 1 1 58FFE010
 P 6750 1900
@@
 $EndComp
 $Comp
-L TEST TP59
+L Connector:TestPoint TP59
 U 1 1 598C15D2
 P 2200 850
@@
 $EndComp
 $Comp
-L TEST TP60
+L Connector:TestPoint TP60
 U 1 1 598C15D3
 P 2400 950
@@
 $EndComp
 $Comp
-L TEST TP71
+L Connector:TestPoint TP71
 U 1 1 598C15D4
 P 5400 4650
@@
 $EndComp
 $Comp
-L TEST TP70
+L Connector:TestPoint TP70
 U 1 1 598C15D5
 P 5350 4350
@@
 $EndComp
 $Comp
-L TEST TP57
+L Connector:TestPoint TP57
 U 1 1 598C15D6
 P 1250 900
@@
 $EndComp
 $Comp
-L TEST TP56
+L Connector:TestPoint TP56
 U 1 1 59765390
 P 1250 800
@@
 $EndComp
 $Comp
-L TEST TP54
+L Connector:TestPoint TP54
 U 1 1 598C15D7
 P 800 2650
@@
 $EndComp
 $Comp
-L TEST TP55
+L Connector:TestPoint TP55
 U 1 1 598C15D8
 P 1000 2500
@@
 $EndComp
 $Comp
-L TEST TP63
+L Connector:TestPoint TP63
 U 1 1 598C15D9
 P 4400 1050
@@
 $EndComp
 $Comp
-L TEST TP66
+L Connector:TestPoint TP66
 U 1 1 598C15DA
 P 4500 1150
@@
 $EndComp
 $Comp
-L TEST TP61
+L Connector:TestPoint TP61
 U 1 1 598C15DB
 P 4250 2450
@@
 $EndComp
 $Comp
-L TEST TP58
+L Connector:TestPoint TP58
 U 1 1 598C15DC
 P 1350 2950
@@
 $EndComp
 $Comp
-L TEST TP64
+L Connector:TestPoint TP64
 U 1 1 598C15DD
 P 4400 2750
@@
 $EndComp
 $Comp
-L TEST TP69
+L Connector:TestPoint TP69
 U 1 1 598C15D1
 P 4600 2650
@@
 $EndComp
 $Comp
-L TEST TP68
+L Connector:TestPoint TP68
 U 1 1 598C15DE
 P 4550 2000
@@
 $EndComp
 $Comp
-L TEST TP67
+L Connector:TestPoint TP67
 U 1 1 598C15DF
 P 4550 1600
@@
 $EndComp
 $Comp
-L TEST TP65
+L Connector:TestPoint TP65
 U 1 1 598C15E0
 P 4450 3150
@@
 RX1
 $Comp
-L TEST TP53
+L Connector:TestPoint TP53
 U 1 1 597B49F7
 P 650 2950
@@
 RX6
 $Comp
-L TEST TP62
+L Connector:TestPoint TP62
 U 1 1 59867FCD
 P 4250 2950
@@
 U4_RX
 $Comp
-L CONN_01X02 J22
+L Connector_Generic:Conn_01x02 J22
 U 1 1 598B52A9
 P 750 1700
@@
 $EndComp
 $Comp
-L TEST_1P J25
+L Connector:TestPoint J25
 U 1 1 598D0D0D
 P 6750 3250
@@
 $EndComp
 $Comp
-L TEST_1P J26
+L Connector:TestPoint J26
 U 1 1 598D0D13
 P 6750 3350
@@
 $EndComp
 $Comp
-L TEST_1P J23
+L Connector:TestPoint J23
 U 1 1 598D1357
 P 6750 3050
@@
 $EndComp
 $Comp
-L TEST_1P J24
+L Connector:TestPoint J24
 U 1 1 598D135D
 P 6750 3150
@@
 $EndSheet
 $Comp
-L TEST_1P J31
+L Connector:TestPoint J31
 U 1 1 5978540F
 P 6750 3900
@@
 $EndComp
 $Comp
-L TEST_1P J32
+L Connector:TestPoint J32
 U 1 1 59785415
 P 6750 4000
@@
 $EndComp
 $Comp
-L TEST_1P J29
+L Connector:TestPoint J29
 U 1 1 5978541B
 P 6750 3700
@@
 $EndComp
 $Comp
-L TEST_1P J30
+L Connector:TestPoint J30
 U 1 1 59785421
 P 6750 3800
@@
 12V
 $Comp
-L TEST_1P J27
+L Connector:TestPoint J27
 U 1 1 598E3B16
 P 6750 3450
@@
 $EndComp
 $Comp
-L TEST_1P J28
+L Connector:TestPoint J28
 U 1 1 598E410B
 P 6750 3550
@@
 $EndComp
 $Comp
-L TEST_1P J33
+L Connector:TestPoint J33
 U 1 1 598E4331
 P 6750 4100
@@
 $EndComp
 $Comp
-L TEST_1P J34
+L Connector:TestPoint J34
 U 1 1 598E4337
 P 6750 4200

Commit message: ESC Center: Upgraded to KiCAD 5.0.1.
Parts:
- C153, C154, C155, C156, C157, C158, C159, C160, C161, C162, C163, C164, C165, C166, C167, C168, C169, C170, C171, C172, C173, C174, C175, C176, C177, C178, C179, C180, C181, C182, C183, C184, C185, C186, C187, C188, C189, C190: symbol C_Small -> Device:C_Small
- D25, D28: symbol D_Small_ALT -> Device:D_Small_ALT
- D26, D27: symbol D_Schottky_Small_ALT -> Device:D_Schottky_Small_ALT
- L13, L14, L15: symbol L_Small -> Device:L_Small
- Q25, Q26: symbol Q_NMOS_DGS -> Device:Q_NMOS_DGS
- R133, R134, R135, R136, R137, R138, R139, R140, R141, R142, R143, R144, R145, R146, R147, R148, R149, R150, R151, R152, R153, R154, R155, R156, R157, R158, R159, R160, R161, R162, R163, R164, R165, R166, R167: symbol R_Small -> Device:R_Small
- U1, U2: symbol TPS54531 -> regul-v2:TPS54531
- U3: symbol LM25116 -> regul-v2:LM25116
Connections:
- wire segments 304 -> 395
Other:
- moved on the sheet: J1, J22, J3, J5, J8
