File: phantom_3_pro_esc_center_board/phantom_3_pro_esc_single.sch (KiCad schematic (older format))
At the start: 103 parts, among them M2 Brushless_Motor_3phase, Q10 AON6504, Q11 AON6504, Q12 AON6504, Q7 AON6504, Q8 AON6504, Q9 AON6504, T2 TMS320F28027F, Y3 ?MHz, Y4 ?MHz

Commit message: ESC Center: Upgraded to KiCAD 5.0.1.
Parts:
- C39, C42, C43, C44, C45, C46, C47, C48, C49, C50, C51, C52, C54, C55, C56, C57, C58, C59, C60, C61, C62, C63, C64, C65, C66, C67, C68, C69: symbol C_Small -> Device:C_Small
- C40, C41, C53, C70, C71, C72, C73, C74, C75, C76: symbol CP1_Small -> Device:CP1_Small
- D10, D12, D7, D8, D9: symbol D_Schottky_Small_ALT -> Device:D_Schottky_Small_ALT
- D11: symbol DRV8301_DCA_56 -> DRV8301_DCA_56_thin:DRV8301_DCA_56
- L4, L5, L6: symbol L -> Device:L
- M2: symbol Brushless_Motor_3phase -> motors:Brushless_Motor_3phase
- Q10, Q11, Q12, Q7, Q8, Q9: symbol Q_NMOS_SDG -> Device:Q_NMOS_SDG
- R34, R35, R36, R37, R38, R39, R40, R41, R42, R43, R44, R45, R46, R47, R48, R49, R50, R61, R63, R65, R66: symbol R -> Device:R
- R51, R52, R53, R54, R55, R56, R57, R58, R59, R60, R62, R64: symbol R_Small -> Device:R_Small
- T2: symbol TMS320F28027F-thin -> texas-uc:TMS320F28027F-thin
- Y3, Y4: symbol Crystal_Small -> Device:Crystal_Small
