File: phantom_3_pro_flight_ctrl_board/phantom_3_pro_flight_ctrl_board.sch (KiCad schematic (older format))
At the start: 46 parts, among them J1 Micro_SD_Card, J8 CONN_MC_FRONT, J9 CONN_MC_BACK, U1 STM32F427II, U2 MS5607, U3 MPU-6500, U5 PA 5xA, U6 RC09

Commit message: Flight Ctrl: Just renamed a symbol library, no real change.
Parts:
- U1: footprint Housings_BGA_custom:BGA-176p25_10x10_11.0x11.0mm_Pitch0.65mm -> Housings_BGA-v2:BGA-176p25_10x10_11.0x11.0mm_Pitch0.65mm
Changed lines of the file:
@@
 F 0 "U1" H 7350 2250 50  0000 C CNN
 F 1 "STM32F427II" H 7350 2350 50  0000 C CNN
-F 2 "Housings_BGA_custom:BGA-176p25_10x10_11.0x11.0mm_Pitch0.65mm" H 7550 2250 60  0001 C CNN
+F 2 "Housings_BGA-v2:BGA-176p25_10x10_11.0x11.0mm_Pitch0.65mm" H 7550 2250 60  0001 C CNN
 F 3 "" H 7550 2150 60  0001 C CNN
 	1    6700 2200
@@
 F 0 "U1" H 1800 2300 50  0000 C CNN
 F 1 "STM32F427II" H 1800 2400 50  0000 C CNN
-F 2 "Housings_BGA_custom:BGA-176p25_10x10_11.0x11.0mm_Pitch0.65mm" H 2000 2300 60  0001 C CNN
+F 2 "Housings_BGA-v2:BGA-176p25_10x10_11.0x11.0mm_Pitch0.65mm" H 2000 2300 60  0001 C CNN
 F 3 "" H 2000 2200 60  0001 C CNN
 	2    1150 2250
@@
 F 0 "U1" H 4350 2300 50  0000 C CNN
 F 1 "STM32F427II" H 4350 2400 50  0000 C CNN
-F 2 "Housings_BGA_custom:BGA-176p25_10x10_11.0x11.0mm_Pitch0.65mm" H 4550 2300 60  0001 C CNN
+F 2 "Housings_BGA-v2:BGA-176p25_10x10_11.0x11.0mm_Pitch0.65mm" H 4550 2300 60  0001 C CNN
 F 3 "" H 4550 2200 60  0001 C CNN
 	3    3700 2250
@@
 F 0 "U1" H 2550 6400 50  0000 C CNN
 F 1 "STM32F427II" H 2550 6500 50  0000 C CNN
-F 2 "Housings_BGA_custom:BGA-176p25_10x10_11.0x11.0mm_Pitch0.65mm" H 2750 6400 60  0001 C CNN
+F 2 "Housings_BGA-v2:BGA-176p25_10x10_11.0x11.0mm_Pitch0.65mm" H 2750 6400 60  0001 C CNN
 F 3 "" H 2750 6300 60  0001 C CNN
 	4    1900 6350

Commit message: All: Preparing for KiCad version change.
Parts:
- J8: symbol CONN_01X20 -> Connector_Generic:Conn_01x20
- J9: symbol CONN_01X21 -> Connector_Generic:Conn_01x21
- J?: symbol CONN_02X12 -> Connector_Generic:Conn_02X12
- TP1, TP10, TP11, TP12, TP13, TP14, TP15, TP16, TP17, TP18, TP19, TP2, TP20, TP3, TP4, TP5, TP6, TP7, TP8, TP9: symbol TEST -> Connector:TestPoint
Other:
- moved on the sheet: TP1, TP10, TP11, TP12, TP13, TP14, TP15, TP16, TP17, TP18, TP19, TP2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
Changed lines of the file:
@@
 $EndDescr
 $Comp
-L CONN_01X20 J8
+L Connector_Generic:Conn_01x20 J8
 U 1 1 58FEFB33
 P 2800 750
@@
 $EndComp
 $Comp
-L CONN_01X21 J9
+L Connector_Generic:Conn_01x21 J9
 U 1 1 58FEFD57
 P 5050 7450
@@
 	9250 2550 9200 2550
 $Comp
-L TEST TP5
+L Connector:TestPoint TP5
 U 1 1 598A06F8
 P 4750 6950
@@
 $EndComp
 $Comp
-L TEST TP4
+L Connector:TestPoint TP4
 U 1 1 598A06F9
 P 3950 7050
@@
 $EndComp
 $Comp
-L TEST TP8
+L Connector:TestPoint TP8
 U 1 1 598A06FA
 P 5950 7000
@@
 $EndComp
 $Comp
-L TEST TP7
+L Connector:TestPoint TP7
 U 1 1 598A06FB
 P 5850 6800
@@
 $EndComp
 $Comp
-L TEST TP20
+L Connector:TestPoint TP20
 U 1 1 598A06FC
 P 10800 5750
@@
 $EndComp
 $Comp
-L TEST TP2
+L Connector:TestPoint TP2
 U 1 1 598A06FD
 P 2550 1450
@@
 $EndComp
 $Comp
-L TEST TP1
+L Connector:TestPoint TP1
 U 1 1 59830F57
 P 2450 1250
@@
 $EndComp
 $Comp
-L TEST TP9
+L Connector:TestPoint TP9
 U 1 1 598A0709
 P 9450 3650
@@
 $EndComp
 $Comp
-L TEST TP11
+L Connector:TestPoint TP11
 U 1 1 598A0708
 P 9750 3650
@@
 $EndComp
 $Comp
-L TEST TP16
+L Connector:TestPoint TP16
 U 1 1 598A0707
 P 10300 3750
@@
 $EndComp
 $Comp
-L TEST TP15
+L Connector:TestPoint TP15
 U 1 1 598A0706
 P 10100 3650
@@
 $EndComp
 $Comp
-L TEST TP10
+L Connector:TestPoint TP10
 U 1 1 598A0705
 P 8600 3700
@@
 $EndComp
 $Comp
-L TEST TP3
+L Connector:TestPoint TP3
 U 1 1 598A0704
 P 3350 6550
@@
 $EndComp
 $Comp
-L TEST TP14
+L Connector:TestPoint TP14
 U 1 1 598A0703
 P 9100 3700
@@
 $EndComp
 $Comp
-L TEST TP12
+L Connector:TestPoint TP12
 U 1 1 598A0702
 P 8850 3700
@@
 $EndComp
 $Comp
-L TEST TP19
+L Connector:TestPoint TP19
 U 1 1 598A0701
 P 10800 3750
@@
 $EndComp
 $Comp
-L TEST TP13
+L Connector:TestPoint TP13
 U 1 1 598A0700
 P 9950 4700
@@
 $EndComp
 $Comp
-L TEST TP17
+L Connector:TestPoint TP17
 U 1 1 598A06FF
 P 10550 3650
@@
 $EndComp
 $Comp
-L TEST TP6
+L Connector:TestPoint TP6
 U 1 1 598A06FE
 P 5150 6950
@@
 $EndComp
 $Comp
-L TEST TP18
+L Connector:TestPoint TP18
 U 1 1 598A06F7
 P 11050 3750
@@
 	5400 1400 5200 1400
 $Comp
-L CONN_02X12 J?
+L Connector_Generic:Conn_02X12 J?
 U 1 1 59900046
 P 9700 1250

Commit message: Flight Ctrl: Upgraded to KiCAD 5.0.1.
Parts:
- removed J1: Micro_SD_Card, Connectors:microSD_Card_Receptacle_Wuerth_693072010801, symbol Micro_SD_Card
- added J1: Micro_SD_Card, symbol Connector:Micro_SD_Card
- C1, C2, C3, C4, C5: symbol C_Small -> Device:C_Small
- J?: symbol Connector_Generic:Conn_02X12 -> Connector_Generic:Conn_02x12_Odd_Even
- R1, R10, R11, R2, R3, R4, R5, R6, R7, R8, R9: symbol R_Small -> Device:R_Small
- U1: symbol STM32F4XXH2 -> texas-uc:STM32F4XXH2
- U2: symbol MS5607_Anno -> sensors-v2:MS5607_Anno
- U3: symbol MPU-6500 -> sensors-v2:MPU-6500
- U5: symbol IC_DIL8 -> ic_dil_generic:IC_DIL8
- U6: symbol IC_SOT5 -> ic_dil_generic:IC_SOT5
- U?: symbol IC_SOT3 -> ic_dil_generic:IC_SOT3
Connections:
- wire segments 149 -> 232
Other:
- moved on the sheet: J8
