File: phantom_3_pro_overview/gimbal_arm_driver.sch (KiCad schematic (older format))
At the start: 0 parts

Commit message: Overview: Work on camera and gimbal.
Parts:
- added Q? (x3): AON7804, Dual N-Ch MOSFET, symbol AON7804-align1
- added RV?: Potentiometer, Motor_Pos_Sense, symbol POT
- added U?: dsPIC33 EP32, motor control sw, symbol IC_PQFP32
- added U? (x3): MP1907, Half-bridge, symbol IC_DIL10
Connections:
- new net: RV?.2, U?.32
- new net: Q?.1 (G1), U?.5 (x3)
- new net: Q?.2 (S1), Q?.4 (D2) (x3)
- new net: Q?.5 (G2), U?.4 (x3)
- new net +BATT: Q?.8 (D1), Q?.8 (D1), Q?.8 (D1), RV?.3, U?.3, U?.3, U?.3
- new net GND: Q?.6 (S2), Q?.6 (S2), Q?.6 (S2), RV?.1, U?.10, U?.10, U?.10

Commit message: Overview: Upgraded to KiCAD 5.0.1.
Parts:
- Q? (x3): symbol AON7804-align1 -> transistors-power:AON7804-align1
- RV?: symbol POT -> Device:R_POT
- U?: symbol IC_PQFP32 -> ic_dil_generic:IC_PQFP32
- U? (x3): symbol IC_DIL10 -> ic_dil_generic:IC_DIL10
Changed lines of the file:
@@
-EESchema Schematic File Version 2
-LIBS:power
-LIBS:device
-LIBS:transistors
-LIBS:conn
-LIBS:linear
-LIBS:regul
-LIBS:74xx
-LIBS:cmos4000
-LIBS:adc-dac
-LIBS:memory
-LIBS:xilinx
-LIBS:microcontrollers
-LIBS:dsp
-LIBS:microchip
-LIBS:analog_switches
-LIBS:motorola
-LIBS:texas
-LIBS:intel
-LIBS:audio
-LIBS:interface
-LIBS:digital-audio
-LIBS:philips
-LIBS:display
-LIBS:cypress
-LIBS:siliconi
-LIBS:opto
-LIBS:atmel
-LIBS:contrib
-LIBS:valves
-LIBS:motors
-LIBS:ic_dil_generic
-LIBS:sensors
-LIBS:u-blox
-LIBS:amplifiers
-LIBS:transistors-switches
-LIBS:transistors-power
-LIBS:sensors-v2
-LIBS:regul-v2
+EESchema Schematic File Version 4
 LIBS:phantom_3_pro_overview-cache
-EELAYER 25 0
+EELAYER 26 0
 EELAYER END
 $Descr User 5197 4724
 encoding utf-8
-Sheet 20 24
+Sheet 21 24
 Title "Overview of the Phantom 3 Pro Gimbal Arm Driver"
 Date ""
@@
 FLAT_MOTOR
 $Comp
-L +BATT #PWR?
+L power:+BATT #PWR?
 U 1 1 5971121C
 P 4100 950
 AR Path="/596E86D9/5971121C" Ref="#PWR?"  Part="1"
 AR Path="/596C09CC/5971121C" Ref="#PWR?"  Part="1"
+AR Path="/596E82ED/5971121C" Ref="#PWR?"  Part="1"
 F 0 "#PWR?" H 4100 800 50  0001 C CNN
 F 1 "+BATT" H 4100 1090 50  0000 C CNN
@@
 $EndComp
 $Comp
-L GND #PWR?
+L power:GND #PWR?
 U 1 1 59711222
 P 4100 1600
 AR Path="/596E86D9/59711222" Ref="#PWR?"  Part="1"
 AR Path="/596C09CC/59711222" Ref="#PWR?"  Part="1"
+AR Path="/596E82ED/59711222" Ref="#PWR?"  Part="1"
 F 0 "#PWR?" H 4100 1350 50  0001 C CNN
 F 1 "GND" H 4100 1450 50  0000 C CNN
@@
 	4150 700  4250 600
 $Comp
-L GND #PWR?
+L power:GND #PWR?
 U 1 1 5971125E
 P 2650 2650
 AR Path="/596E86D9/5971125E" Ref="#PWR?"  Part="1"
 AR Path="/596C09CC/5971125E" Ref="#PWR?"  Part="1"
+AR Path="/596E82ED/5971125E" Ref="#PWR?"  Part="1"
 F 0 "#PWR?" H 2650 2400 50  0001 C CNN
 F 1 "GND" H 2650 2500 50  0000 C CNN
@@
 $EndComp
 $Comp
-L +BATT #PWR?
+L power:+BATT #PWR?
 U 1 1 59711264
 P 2450 1850
 AR Path="/596E86D9/59711264" Ref="#PWR?"  Part="1"
 AR Path="/596C09CC/59711264" Ref="#PWR?"  Part="1"
+AR Path="/596E82ED/59711264" Ref="#PWR?"  Part="1"
 F 0 "#PWR?" H 2450 1700 50  0001 C CNN
 F 1 "+BATT" H 2450 1990 50  0000 C CNN
@@
 	2000 2750 2100 2850
 $Comp
-L IC_PQFP32 U?
+L ic_dil_generic:IC_PQFP32 U?
 U 1 1 597112C4
 P 1300 2150
 AR Path="/596E86D9/597112C4" Ref="U?"  Part="1"
 AR Path="/596C09CC/597112C4" Ref="U?"  Part="1"
+AR Path="/596E82ED/597112C4" Ref="U?"  Part="1"
 F 0 "U?" H 1300 2050 50  0001 C CNN
 F 1 "dsPIC33 EP32" H 1300 2250 50  0000 C CNN
@@
 	1900 1450 2000 1550
 $Comp
-L AON7804-align1 Q?
+L transistors-power:AON7804-align1 Q?
 U 1 1 59714F5F
 P 3900 1250
 AR Path="/596E86D9/59714F5F" Ref="Q?"  Part="1"
 AR Path="/596C09CC/59714F5F" Ref="Q?"  Part="1"
+AR Path="/596E82ED/59714F5F" Ref="Q?"  Part="1"
 F 0 "Q?" H 3650 1025 50  0001 L CNN
 F 1 "AON7804" H 3700 1000 50  0000 L CNN
@@
 $EndComp
 $Comp
-L +BATT #PWR?
+L power:+BATT #PWR?
 U 1 1 59716694
 P 3450 950
@@
 $EndComp
 $Comp
-L GND #PWR?
+L power:GND #PWR?
 U 1 1 5971669A
 P 3450 1600
@@
 	3500 700  3600 600
 $Comp
-L AON7804-align1 Q?
+L transistors-power:AON7804-align1 Q?
 U 1 1 597166A6
 P 3250 1250
@@
 $EndComp
 $Comp
-L +BATT #PWR?
+L power:+BATT #PWR?
 U 1 1 597166B3
 P 2800 950
@@
 $EndComp
 $Comp
-L GND #PWR?
+L power:GND #PWR?
 U 1 1 597166B9
 P 2800 1600
@@
 	2850 700  2950 600
 $Comp
-L AON7804-align1 Q?
+L transistors-power:AON7804-align1 Q?
 U 1 1 597166C5
 P 2600 1250
@@
 $EndComp
 $Comp
-L IC_DIL10 U?
+L ic_dil_generic:IC_DIL10 U?
 U 1 1 59716CA5
 P 2450 2250
 AR Path="/596E86D9/59716CA5" Ref="U?"  Part="1"
 AR Path="/596C09CC/59716CA5" Ref="U?"  Part="1"
+AR Path="/596E82ED/59716CA5" Ref="U?"  Part="1"
 F 0 "U?" H 2450 2150 50  0001 C CNN
 F 1 "MP1907" H 2450 2350 50  0000 C CNN
@@
 Wire Wire Line
 	750  2500 700  2500
-Wire Bus Line
-	2950 600  4300 600
 Wire Wire Line
 	950  2700 950  2750
@@
 Wire Wire Line
 	750  2100 700  2100
-Wire Bus Line
-	700  2850 3750 2850
-Wire Bus Line
-	1150 1450 1900 1450
-Wire Bus Line
-	2000 1550 2000 2750
-Wire Bus Line
-	600  1800 600  2750
 Wire Wire Line
 	4100 1050 4100 950
 Wire Wire Line
-	4100 1200 4100 1300
+	4100 1200 4100 1250
 Wire Wire Line
 	4100 1450 4100 1600
@@
 	3450 1050 3450 950
 Wire Wire Line
-	3450 1200 3450 1300
+	3450 1200 3450 1250
 Wire Wire Line
 	3450 1450 3450 1600
@@
 	2800 1050 2800 950
 Wire Wire Line
-	2800 1200 2800 1300
+	2800 1200 2800 1250
 Wire Wire Line
 	2800 1450 2800 1600
@@
 	2250 1150 2350 1150
 $Comp
-L GND #PWR?
+L power:GND #PWR?
 U 1 1 597170ED
 P 3300 2650
 AR Path="/596E86D9/597170ED" Ref="#PWR?"  Part="1"
 AR Path="/596C09CC/597170ED" Ref="#PWR?"  Part="1"
+AR Path="/596E82ED/597170ED" Ref="#PWR?"  Part="1"
 F 0 "#PWR?" H 3300 2400 50  0001 C CNN
 F 1 "GND" H 3300 2500 50  0000 C CNN
@@
 $EndComp
 $Comp
-L IC_DIL10 U?
+L ic_dil_generic:IC_DIL10 U?
 U 1 1 597170F3
 P 3100 2250
@@
 $EndComp
 $Comp
-L GND #PWR?
+L power:GND #PWR?
 U 1 1 597170F9
 P 3950 2650
 AR Path="/596E86D9/597170F9" Ref="#PWR?"  Part="1"
 AR Path="/596C09CC/597170F9" Ref="#PWR?"  Part="1"
+AR Path="/596E82ED/597170F9" Ref="#PWR?"  Part="1"
 F 0 "#PWR?" H 3950 2400 50  0001 C CNN
 F 1 "GND" H 3950 2500 50  0000 C CNN
@@
 $EndComp
 $Comp
-L IC_DIL10 U?
+L ic_dil_generic:IC_DIL10 U?
 U 1 1 597170FF
 P 3750 2250
@@
 $EndComp
 $Comp
-L +BATT #PWR?
+L power:+BATT #PWR?
 U 1 1 59717111
 P 3100 1850
 AR Path="/596E86D9/59717111" Ref="#PWR?"  Part="1"
 AR Path="/596C09CC/59717111" Ref="#PWR?"  Part="1"
+AR Path="/596E82ED/59717111" Ref="#PWR?"  Part="1"
 F 0 "#PWR?" H 3100 1700 50  0001 C CNN
 F 1 "+BATT" H 3100 1990 50  0000 C CNN
@@
 $EndComp
 $Comp
-L +BATT #PWR?
+L power:+BATT #PWR?
 U 1 1 59717125
 P 3750 1850
 AR Path="/596E86D9/59717125" Ref="#PWR?"  Part="1"
 AR Path="/596C09CC/59717125" Ref="#PWR?"  Part="1"
+AR Path="/596E82ED/59717125" Ref="#PWR?"  Part="1"
 F 0 "#PWR?" H 3750 1700 50  0001 C CNN
 F 1 "+BATT" H 3750 1990 50  0000 C CNN
@@
 	4300 600  4300 650
 $Comp
-L POT RV?
+L Device:R_POT RV?
 U 1 1 59717774
 P 1350 1000
 AR Path="/596E86D9/59717774" Ref="RV?"  Part="1"
 AR Path="/596C09CC/59717774" Ref="RV?"  Part="1"
+AR Path="/596E82ED/59717774" Ref="RV?"  Part="1"
 F 0 "RV?" V 1175 1000 50  0001 C CNN
 F 1 "Potentiometer" V 1200 1000 50  0000 C CNN
@@
 $EndComp
 $Comp
-L +BATT #PWR?
+L power:+BATT #PWR?
 U 1 1 5971780C
 P 1350 850
 AR Path="/596E86D9/5971780C" Ref="#PWR?"  Part="1"
 AR Path="/596C09CC/5971780C" Ref="#PWR?"  Part="1"
+AR Path="/596E82ED/5971780C" Ref="#PWR?"  Part="1"
 F 0 "#PWR?" H 1350 700 50  0001 C CNN
 F 1 "+BATT" H 1350 990 50  0000 C CNN
@@
 $EndComp
 $Comp
-L GND #PWR?
+L power:GND #PWR?
 U 1 1 59717821
 P 1350 1150
@@
 Wire Wire Line
 	950  1000 1200 1000
+Wire Wire Line
+	4100 1250 4100 1300
+Wire Wire Line
+	3450 1250 3450 1300
+Wire Wire Line
+	2800 1250 2800 1300
+Wire Bus Line
+	2950 600  4300 600
+Wire Bus Line
+	1150 1450 1900 1450
+Wire Bus Line
+	600  1800 600  2750
+Wire Bus Line
+	2000 1550 2000 2750
+Wire Bus Line
+	700  2850 3750 2850
 $EndSCHEMATC

Commit message: All: Finished updating to KiCad 5.0.1.
Parts:
- Q? (x3): symbol transistors-power:AON7804-align1 -> Transistor_FET-v2:AON7804-align1
Changed lines of the file:
@@
 	1900 1450 2000 1550
 $Comp
-L transistors-power:AON7804-align1 Q?
+L Transistor_FET-v2:AON7804-align1 Q?
 U 1 1 59714F5F
 P 3900 1250
@@
 	3500 700  3600 600
 $Comp
-L transistors-power:AON7804-align1 Q?
+L Transistor_FET-v2:AON7804-align1 Q?
 U 1 1 597166A6
 P 3250 1250
@@
 	2850 700  2950 600
 $Comp
-L transistors-power:AON7804-align1 Q?
+L Transistor_FET-v2:AON7804-align1 Q?
 U 1 1 597166C5
 P 2600 1250
